File: FIPI_shematics.sch (EAGLE design)
At the start: 21 parts, among them IC1 LM324D, IC2 7805DT

Commit message: FIPI_schematics
Parts:
- removed IC1: LM324D, linear:LM324D
- removed U$2: MALE_HEADER, male_header_device:MALE_HEADER
- added C10, C11, C6, C7, C8, C9: 0.1u, rcl:C-EUC1206
- added C12, C13, C14, C15: 10u, rcl:C-EUC1206
- added C5: 100u, rcl:C-EUC1206
- added D1: 1N4007, casovac:1N4007
- added IC3: FT232RL, ftdichip:FT232RL
- added IC4: MAX202CSE, maxim-8:MAX202CSE
- added IC5, IC6: MCP23017SO, adafruit:MCP23017SO
- added LED1, LED2: (no value), eagle-ltspice:LED_E
- added R12, R13: 270E, resistor:R-EU_R1206
- added RASPPI: MALE_HEADER, male_header_device:MALE_HEADER
- added SW1: (no value), adafruit:SWITCH_PUSHBUTTONSOFTTOUCHSMD_SJ
- added U$4: SWITCH1, switch:SWITCH1
- added U$5: PORT_EXP, fem_header:PORT_EXP
- added U$7: SERVO, switch:SERVO
- added U1, U2, U3: MCP3008-I/SL, MCP3008-I_SL:MCP3008-I/SL
- added U4: (no value), SparkFun-IC-Power:V_REG_LM1117SOT223
- added U5: LMV324, SparkFun-IC-Amplifiers:LMV324
- IC2: value 7805DT -> (none); device linear:7805DT -> tango:L7805
- U$3: value SWITCH -> SWITCH_RXTX; device switch:SWITCH -> switch:SWITCH_RXTX
Connections:
- removed net 5V-SYS1: R3.1, U$1.P10
- removed net 5V-SYS2: U$1.P7
- removed net N$10: IC1B.OUT, U$3.5, U$3.6, U$3.7
- removed net N$11: IC1C.OUT, U$3.3, U$3.4
- removed net N$12: IC1D.OUT, U$3.1, U$3.2
- removed net N$13: D2.A, U$3.1"
- removed net N$18: D2.A5, U$3.6"
- new net 3.3V: IC5.!RESET, IC5.VDD, IC6.!RESET, IC6.A0, IC6.VDD, RASPPI.3.3-2, RASPPI.3.31, U$5.40, U1.VDD, U1.VREF, U2.VDD, U2.VREF, U3.VDD, U3.VREF
- new net 5V: C10.2, C11.2, IC4.VCC, R3.1, SW1.P$2, U$1.P7, U$5.1, U5G5.P$V+
- new net 5V_SERVO: C13.1, C14.1, U$7.1, U$7.1", U$7.1', U4.OUT
- new net BARGRAPH1: D2.A, IC5.GPB2
- new net BARGRAPH2: D2.A1, IC5.GPB3
- new net BARGRAPH3: D2.A2, IC5.GPB4
- new net BARGRAPH4: D2.A3, IC5.GPB5
- new net BARGRAPH5: D2.A4, IC5.GPB6
- new net BUZZER: IC5.GPA6, U$1.71
- new net CE0: RASPPI.CE0, U1.*CS/SHDN
- new net CE1: RASPPI.CE1, U2.*CS/SHDN
- new net CE2: RASPPI.25, U3.*CS/SHDN
- new net DB4: RASPPI.13, U$1.26
- new net DB5: RASPPI.6, U$1.25
- new net DB6: RASPPI.5, U$1.27
- new net DB7: RASPPI.21, U$1.28
- new net EN: RASPPI.19, U$1.24
- new net INTERRUPT: RASPPI.4, SW1.P$1
- new net IRP1: U$1.P12, U1.CH2
- new net IRP2: U$1.P16, U1.CH0
- new net IRP3: U$1.42, U2.CH4
- new net IRP4: U$1.43, U2.CH5
- new net IRP5: U$1.46, U1.CH7
- new net IRP6: U$1.69, U3.CH0
- new net IRP7: U$1.70, U3.CH1
- new net IRP8: U$1.P2, U1.CH4
- new net IRPD: RASPPI.16, U$1.34
- new net L1: IC5.GPA1, U$1.51
- new net L2: IC5.GPA2, U$1.52
- new net MB73: IC4.R1IN, U$1.73
- new net MB74: IC4.T1OUT, U$1.74
- new net MISO: RASPPI.9, U$5.37, U1.DOUT, U2.DOUT, U3.DOUT
- new net MOSI: RASPPI.10, U$5.36, U1.DIN, U2.DIN, U3.DIN
- new net N$23: IC3.CBUS0, LED1.A
- new net N$24: IC3.CBUS1, LED2.A
- new net N$25: LED1.C, R12.1
- new net N$26: LED2.C, R13.1
- new net PEL: RASPPI.24, U$1.62
- new net PER: RASPPI.23, U$1.63
- new net PWML: IC5.GPA0, U$1.50
- new net PWMR: IC5.GPA4, U$1.54
- new net R1: IC5.GPA3, U$1.53
- new net R2: IC5.GPA5, U$1.55
- new net RS: RASPPI.26, U$1.22
- new net RX: RASPPI.TX, U$3.1'
- new net RXFT: IC3.RXD, U$3.2'
- new net RXP: U$3.5', U$5.30
- new net RXRS: IC4.R1OUT, U$3.4'
- new net RXXB: U$1.P13, U$3.3'
- new net SCL: IC5.SCL, IC6.SCL, RASPPI.SCL, U$5.28
- new net SCLK: RASPPI.11, U$5.38, U1.CLK, U2.CLK, U3.CLK
- new net SDA: IC5.SDA, IC6.SDA, RASPPI.SDA, U$5.27
- new net SERVO1: IC5.GPA7, RASPPI.17, U$7.2
- new net SERVO2: IC5.GPB0, RASPPI.27, U$7.2'
- new net SERVO3: IC5.GPB1, RASPPI.22, U$7.2"
- new net SIR1: U$1.P11, U1.CH3
- new net SIR2: U$1.P15, U1.CH1
- new net SIR3: U$1.41, U2.CH3
- new net SIR4: U$1.44, U2.CH6
- new net SIR5: U$1.45, U2.CH7
- new net SIRD: RASPPI.12, U$1.33
- new net TSOP: U1.CH6
- new net TX: RASPPI.RX, U$3.1
- new net TXFT: IC3.TXD, U$3.2
- new net TXP: U$3.5, U$5.29
- new net TXRS: IC4.T1IN, U$3.4
- new net TXXB: U$1.P14, U$3.3
- new net USB+: IC3.USBDP, U$1.P4
- new net USB-: IC3.USBDM, U$1.P5
- new net V+: C10.1, IC4.V+
- new net V-: C7.1, IC4.V-
- new net VOLT_SENS: C1.2, C2.1, R1.2, R2.1, U1.CH5, U5G1.+IN, U5G2.+IN, U5G3.+IN, U5G4.+IN
- new net VUSB: C5.1, C6.1, IC3.VCC, IC3.VCCIO, U$1.P6
- new net WLS1: U$1.30, U2.CH0
- new net WLS2: U$1.31, U2.CH1
- new net WLS3: U$1.32, U2.CH2
- new net WLS4: U$5.35
- new net WLS5: U$5.34
- new net WLS6: U$5.31
- new net WLS7: U$5.32
- new net WLSD: RASPPI.20, U$1.40
- new net XADC1: U$5.2, U3.CH2
- new net XADC2: U$5.3, U3.CH3
- new net XADC3: U$5.4, U3.CH4
- new net XADC4: U$5.5, U3.CH5
- new net XADC5: U$5.6, U3.CH6
- new net XADC6: U$5.7, U3.CH7
- new net XGPIO1: IC5.GPB7, U$5.8
- new net XGPIO10: IC6.GPB0, U$5.17
- new net XGPIO11: IC6.GPB1, U$5.18
- new net XGPIO12: IC6.GPB2, U$5.19
- new net XGPIO13: IC6.GPB3, U$5.22
- new net XGPIO14: IC6.GPB4, U$5.23
- new net XGPIO15: IC6.GPB5, U$5.24
- new net XGPIO16: IC6.GPB6, U$5.25
- new net XGPIO17: IC6.GPB7, U$5.26
- new net XGPIO2: IC6.GPA0, U$5.9
- new net XGPIO3: IC6.GPA1, U$5.10
- new net XGPIO4: IC6.GPA2, U$5.11
- new net XGPIO5: IC6.GPA3, U$5.12
- new net XGPIO6: IC6.GPA4, U$5.13
- new net XGPIO7: IC6.GPA5, U$5.14
- new net XGPIO8: IC6.GPA6, U$5.15
- new net XGPIO9: IC6.GPA7, U$5.16
- net 9-12V: now also D1.A, IC2.IN, U$5.33, U$5.39; no longer IC2.VI
- net GND: now also C11.1, C12.2, C13.2, C14.2, C15.2, C5.2, C6.2, C7.2, IC3.GND, IC3.GND@1, IC3.GND@2, IC3.GND@A, IC3.TEST, IC4.GND, IC5.A0, IC5.A1, IC5.A2, IC5.VSS, IC6.A1, IC6.A2, IC6.VSS, R12.2, R13.2, RASPPI.GND1, RASPPI.GND3, RASPPI.GND6, RASPPI.GND7, RASPPI.GND8, U$1.23, U$4.1, U$5.20, U$5.21, U$7.3, U$7.3", U$7.3', U1.AGND, U1.DGND, U2.AGND, U2.DGND, U3.AGND, U3.DGND, U4.ADJ, U5G5.P$V-; no longer D2.C5, D2.C6, D2.C7, D2.C8, D2.C9, U$2.GND1
- net N$14: now also D2.A8, D2.A9, U5G4.OUT; no longer D2.A1, U$3.2"
- net N$15: now also D2.A7, U5G2.OUT; no longer D2.A2, U$3.3"
- net N$16: now also D2.A6, U5G3.OUT; no longer D2.A3, U$3.4"
- net N$17: now also D2.A5, U5G1.OUT; no longer D2.A4, U$3.5"
- net N$19: now also C8.1, IC4.C1+; no longer D2.A6, U$3.7"
- net N$2: now also C12.1, C15.1, D1.C, U4.IN; no longer C1.2, C2.1, IC1A.+IN, IC1B.+IN, IC1C.+IN, IC1D.+IN, R1.2, R2.1
- net N$20: now also C8.2, IC4.C1-; no longer D2.A7, U$3.8"
- net N$21: now also C9.1, IC4.C2+; no longer D2.A8, U$3.9"
- net N$22: now also C9.2, IC4.C2-; no longer D2.A9, U$3.10"
- net N$3: now also U5G1.-IN; no longer IC1A.-IN
- net N$6: now also U5G3.-IN; no longer IC1B.-IN
- net N$7: now also U5G2.-IN; no longer IC1C.-IN
- net N$8: now also U5G4.-IN; no longer IC1D.-IN
- net N$9: now also D2.C5, D2.C6, D2.C7, D2.C8, D2.C9, U$4.2; no longer IC1A.OUT, U$3.10, U$3.8, U$3.9
- net RASP_5V: now also IC2.OUT, RASPPI.5-1; no longer IC2.VO, U$2.5-1
Other:
- moved on the sheet: C1, C2, C3, C4, D2, R1, R10, R11, R2, R3, R4, R5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
